File: redox-w/pcb/redox_w_transmitters_kicad_files/redox_rev1.sch (KiCad schematic (older format))
At the start: 91 parts, among them K0 KEYSW, K1 KEYSW, K10 KEYSW, K11 KEYSW, K12 KEYSW, K13 KEYSW, K14 KEYSW, K15 KEYSW, K16 KEYSW, K2 KEYSW, K20 KEYSW, K21 KEYSW, K22 KEYSW, K23 KEYSW, K24 KEYSW, K25 KEYSW, K26 KEYSW, K3 KEYSW, K30 KEYSW, K31 KEYSW, K32 KEYSW, K33 KEYSW, K34 KEYSW, K35 KEYSW, K36 KEYSW, K4 KEYSW, K40 KEYSW, K41 KEYSW, K42 KEYSW, K43 KEYSW, K44 KEYSW, K45 KEYSW, K46 KEYSW, K5 KEYSW, K6 KEYSW, Q1 DMG2301L

Commit message: WIP - Right Before PCB Update
Parts:
- BT_LEFT1: renamed from BT_RIGHT?; value Battery_Cell -> Battery_Cel; footprint Battery:BatteryHolder_Keystone_3034_1x20mm -> redox_w_footprints:BatteryHolder_Keystone_3034_1x20mm
- BT_RIGHT1: footprint Battery:BatteryHolder_Keystone_3034_1x20mm -> redox_w_footprints:BatteryHolder_Keystone_3034_1x20mm
- C_LEFT1, C_RIGHT1: renamed from C1; footprint (none) -> Capacitor_SMD:C_0805_2012Metric_Pad1.15x1.40mm_HandSolder
- D0, D1, D10, D11, D12, D13, D14, D15, D16, D2, D20, D21, D22, D23, D24, D25, D26, D3, D30, D31, D32, D33, D34, D35, D36, D4, D40, D41, D42, D43, D44, D45, D46, D5, D6: footprint Keebio-Parts:Diode-dual -> redox_w_footprints:Diode-dual
- JP_LEFT1, JP_RIGHT1: renamed from JP1; footprint (none) -> Jumper:SolderJumper-2_P1.3mm_Bridged2Bar_Pad1.0x1.5mm
- JP_LEFT2, JP_RIGHT2: renamed from JP2; footprint (none) -> Jumper:SolderJumper-2_P1.3mm_Bridged2Bar_Pad1.0x1.5mm
- J_PROG_PORT1: footprint Connector_PinHeader_2.54mm:PinHeader_1x04_P2.54mm_Vertical -> redox_w_footprints:PinHeader_1x04_P2.54mm_Horizontal
- K0, K10, K20, K30, K44: footprint Keebio-Parts:Hybrid_PCB_100H_Dual_hole-nosilk -> redox_w_footprints:Mx_Alps_125-dualside
- K1, K11, K12, K13, K14, K15, K2, K21, K22, K23, K24, K25, K26, K3, K31, K32, K33, K34, K35, K36, K4, K40, K41, K42, K43, K5, K6: footprint Keebio-Parts:Hybrid_PCB_100H_Dual_hole-nosilk -> redox_w_footprints:Mx_Alps_100-dualside
- K16, K45, K46: footprint Keebio-Parts:Hybrid_PCB_100H_Dual_hole-nosilk -> redox_w_footprints:Mx_Alps_150-dualside
- R1, R2: footprint (none) -> Resistor_SMD:R_0805_2012Metric_Pad1.15x1.40mm_HandSolder
- SW_LEFT1: renamed from SW_RIGHT?; footprint Button_Switch_SMD:SW_SPDT_CK-JS102011SAQN -> redox_w_footprints:SW_SPDT_CK-JS102011SAQN
- SW_RIGHT1: footprint Button_Switch_SMD:SW_SPDT_CK-JS102011SAQN -> redox_w_footprints:SW_SPDT_CK-JS102011SAQN
- TRRS1: footprint (none) -> redox_w_footprints:TRRS-PJ-320A-dual
- U_LEFT1, U_RIGHT1: footprint YJ-14015:YJ-14015-Modul -> redox_w_footprints:MY-YJ-14015-Module
- U_RIGHT2: footprint (none) -> redox_w_footprints:ArduinoProMicro
- renumbered Q1 to Q_LEFT1, Q1 to Q_RIGHT1

Commit message: Finished Placing Power Circuitry On PCB
Parts:
- BT_LEFT1: value Battery_Cel -> Battery_Cell
Changed lines of the file:
@@
 P 7100 5850
 F 0 "BT_LEFT1" H 7218 5946 50  0000 L CNN
-F 1 "Battery_Cel" H 7218 5855 50  0000 L CNN
+F 1 "Battery_Cell" H 7218 5855 50  0000 L CNN
 F 2 "redox_w_footprints:BatteryHolder_Keystone_3034_1x20mm" V 7100 5910 50  0001 C CNN
 F 3 "~" V 7100 5910 50  0001 C CNN

Commit message: wip
Parts:
- removed C_LEFT1, C_RIGHT1: 1 μF, Capacitor_SMD:C_0805_2012Metric_Pad1.15x1.40mm_HandSolder, symbol Device:C
- removed JP_LEFT1, JP_RIGHT2: SolderJumper_2_Bridged, Jumper:SolderJumper-2_P1.3mm_Bridged2Bar_Pad1.0x1.5mm, symbol Jumper:SolderJumper_2_Bridged
- removed JP_LEFT2, JP_RIGHT1: SolderJumper_2_Open, Jumper:SolderJumper-2_P1.3mm_Bridged2Bar_Pad1.0x1.5mm, symbol Jumper:SolderJumper_2_Open
- added C_1: 1 μF, Capacitor_SMD:C_0805_2012Metric_Pad1.15x1.40mm_HandSolder, symbol Device:C
- added R3: 4.7k, Resistor_SMD:R_0805_2012Metric_Pad1.15x1.40mm_HandSolder, symbol Device:R
- renumbered U_RIGHT2 to U_LEFT3, U_RIGHT3 to U_RIGHT2
Connections:
- net VCC1 is gone; now on net VCC: TRRS1.1
- net GND: now also C_1.2
- net VCC: now also C_1.1, R3.1
- net ON_BATT: now reaches U_RIGHT1.21 (P07)
- net ON_BATT: now also U_LEFT1.16 (P02), U_LEFT2.4 (STAT), U_RIGHT2.4 (STAT), R3.2
- no-connect marks 52 -> 48
Other:
- moved on the sheet: BT_LEFT1, BT_RIGHT1, Q_LEFT1, Q_RIGHT1, SW_LEFT1, SW_RIGHT1, U_LEFT2, U_LEFT3, U_RIGHT2
