File: redox-w/pcb/redox_w_transmitters_kicad_files/_autosave-redox_rev1.sch (KiCad schematic (older format))
At the start: 85 parts, among them K0 KEYSW, K1 KEYSW, K10 KEYSW, K11 KEYSW, K12 KEYSW, K13 KEYSW, K14 KEYSW, K15 KEYSW, K16 KEYSW, K2 KEYSW, K20 KEYSW, K21 KEYSW, K22 KEYSW, K23 KEYSW, K24 KEYSW, K25 KEYSW, K26 KEYSW, K3 KEYSW, K30 KEYSW, K31 KEYSW, K32 KEYSW, K33 KEYSW, K34 KEYSW, K35 KEYSW, K36 KEYSW, K4 KEYSW, K40 KEYSW, K41 KEYSW, K42 KEYSW, K43 KEYSW, K44 KEYSW, K45 KEYSW, K46 KEYSW, K5 KEYSW, K6 KEYSW

Commit message: Roughly Finished PCB - Changed To Not Mirror Power Circuit
Other:
- moved on the sheet: C_1
Changed lines of the file:
@@
 	0    1    -1   0
 $EndComp
-Wire Wire Line
-	6050 5000 6050 4850
-Connection ~ 6050 5000
-Wire Wire Line
-	6050 5150 6050 5000
 $Comp
 L power:GND #PWR0110
 U 1 1 5EA69E1C
-P 5750 5000
-F 0 "#PWR0110" H 5750 4750 50  0001 C CNN
-F 1 "GND" V 5755 4872 50  0000 R CNN
-F 2 "" H 5750 5000 50  0001 C CNN
-F 3 "" H 5750 5000 50  0001 C CNN
-	1    5750 5000
+P 5750 4850
+F 0 "#PWR0110" H 5750 4600 50  0001 C CNN
+F 1 "GND" V 5755 4722 50  0000 R CNN
+F 2 "" H 5750 4850 50  0001 C CNN
+F 3 "" H 5750 4850 50  0001 C CNN
+	1    5750 4850
 	0    1    -1   0
 $EndComp
@@
 L Device:C C_1
 U 1 1 5EA69E16
-P 5900 5000
-F 0 "C_1" V 5750 5000 50  0000 C CNN
-F 1 "1 μF" V 5650 5000 50  0000 C CNN
-F 2 "Capacitor_SMD:C_0805_2012Metric_Pad1.15x1.40mm_HandSolder" H 5938 4850 50  0001 C CNN
-F 3 "~" H 5900 5000 50  0001 C CNN
-	1    5900 5000
+P 5900 4850
+F 0 "C_1" V 5750 4850 50  0000 C CNN
+F 1 "1 μF" V 5650 4850 50  0000 C CNN
+F 2 "Capacitor_SMD:C_0805_2012Metric_Pad1.15x1.40mm_HandSolder" H 5938 4700 50  0001 C CNN
+F 3 "~" H 5900 4850 50  0001 C CNN
+	1    5900 4850
 	0    1    -1   0
 $EndComp
@@
 $EndComp
 $Comp
-L power:VCC #PWR?
+L power:VCC #PWR0112
 U 1 1 5E8D360D
 P 6100 6250
-F 0 "#PWR?" H 6100 6100 50  0001 C CNN
+F 0 "#PWR0112" H 6100 6100 50  0001 C CNN
 F 1 "VCC" H 6118 6423 50  0000 C CNN
 F 2 "" H 6100 6250 50  0001 C CNN
@@
 	8900 5150 8900 5350
 Connection ~ 8300 5150
+Connection ~ 6050 4850
+Wire Wire Line
+	6050 4850 6050 5150
 $EndSCHEMATC
